File: controls.kicad_sch (KiCad schematic)
At the start: 29 parts, among them J10 IN 1x6h, J11 SYNC, J12 PWM, J13 CV, J14 1VOct, J15 FM, J17 OCT_SW 1x7h, J19 CV 1x6h, J2 SQR, J21 LED 1x2h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

Commit message: Added fp and moved controls
Parts:
- D1: footprint (none) -> LED_THT:LED_D3.0mm_FlatTop
- H5, H6, H7, H8: value ~ -> (none)
- J21: footprint (none) -> Connector_PinHeader_2.54mm:PinHeader_1x02_P2.54mm_Vertical
- J7: footprint (none) -> Connector_PinHeader_2.54mm:PinHeader_1x08_P2.54mm_Vertical

Commit message: Designed PCB and generated JLCPCB files
Parts:
- removed J17: OCT_SW 1x7h, Connector_PinHeader_2.54mm:PinHeader_1x07_P2.54mm_Vertical, symbol Connector:Conn_01x07_Pin
- added J22: OCT 1x6h, Connector_PinHeader_2.54mm:PinHeader_1x06_P2.54mm_Vertical, symbol Connector:Conn_01x06_Pin
Connections:
- net GND: now also SW2.6
- net at SW2.1: now also J22.1 (Pin_1)
- net at SW2.2: now also J22.2 (Pin_2)
- net at SW2.3: now also J22.3 (Pin_3)
- net at SW2.4: now also J22.4 (Pin_4)
- net at SW2.5: now also J22.5 (Pin_5)
- net at SW2.7: now also J22.6 (Pin_6)
Changed lines of the file:
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@@
 	(wire
 		(pts
+			(xy 118.11 63.5) (xy 118.11 66.04)
+		)
+		(stroke
+			(width 0)
+			(type default)
+		)
+	)
+	(wire
+		(pts
 			(xy 251.46 96.52) (xy 266.7 96.52)
 		)
@@
 	(wire
 		(pts
-			(xy 107.95 63.5) (xy 120.65 63.5)
+			(xy 129.54 120.65) (xy 129.54 129.54)
 		)
 		(stroke
@@
 	(wire
 		(pts
-			(xy 129.54 120.65) (xy 129.54 129.54)
+			(xy 107.95 63.5) (xy 113.03 63.5)
 		)
 		(stroke
@@
 	(wire
 		(pts
+			(xy 113.03 72.39) (xy 138.43 72.39)
+		)
+		(stroke
+			(width 0)
+			(type default)
+		)
+	)
+	(wire
+		(pts
 			(xy 114.3 101.6) (xy 106.68 101.6)
 		)
@@
 	(wire
 		(pts
-			(xy 107.95 66.04) (xy 138.43 66.04)
-		)
-		(stroke
-			(width 0)
-			(type default)
-		)
-	)
-	(wire
-		(pts
 			(xy 30.48 113.03) (xy 41.91 113.03)
 		)
@@
 	(wire
 		(pts
+			(xy 120.65 63.5) (xy 118.11 63.5)
+		)
+		(stroke
+			(width 0)
+			(type default)
+		)
+	)
+	(wire
+		(pts
 			(xy 78.74 80.01) (xy 64.77 80.01)
 		)
@@
 	(wire
 		(pts
-			(xy 138.43 58.42) (xy 138.43 66.04)
+			(xy 245.11 83.82) (xy 248.92 83.82)
 		)
 		(stroke
@@
 	(wire
 		(pts
-			(xy 245.11 83.82) (xy 248.92 83.82)
+			(xy 193.04 107.95) (xy 186.69 107.95)
 		)
 		(stroke
@@
 	(wire
 		(pts
-			(xy 193.04 107.95) (xy 186.69 107.95)
+			(xy 179.07 87.63) (xy 186.69 87.63)
 		)
 		(stroke
@@
 	(wire
 		(pts
-			(xy 179.07 87.63) (xy 186.69 87.63)
+			(xy 205.74 90.17) (xy 191.77 90.17)
 		)
 		(stroke
@@
 	(wire
 		(pts
-			(xy 205.74 90.17) (xy 191.77 90.17)
+			(xy 186.69 87.63) (xy 186.69 107.95)
 		)
 		(stroke
@@
 	(wire
 		(pts
-			(xy 186.69 87.63) (xy 186.69 107.95)
+			(xy 132.08 111.76) (xy 137.16 111.76)
 		)
 		(stroke
@@
 	(wire
 		(pts
-			(xy 132.08 111.76) (xy 137.16 111.76)
+			(xy 138.43 58.42) (xy 138.43 72.39)
 		)
 		(stroke
@@
 		)
 	)
+	(wire
+		(pts
+			(xy 113.03 63.5) (xy 113.03 72.39)
+		)
+		(stroke
+			(width 0)
+			(type default)
+		)
+	)
 	(symbol
 		(lib_id "Connector_Audio:AudioJack2_SwitchT")
@@
 	)
 	(symbol
+		(lib_id "Connector:Conn_01x06_Pin")
+		(at 102.87 55.88 0)
+		(unit 1)
+		(body_style 1)
+		(exclude_from_sim no)
+		(in_bom yes)
+		(on_board yes)
+		(in_pos_files yes)
+		(dnp no)
+		(fields_autoplaced yes)
+		(property "Reference" "J22"
+			(at 103.505 45.72 0)
+			(show_name no)
+			(do_not_autoplace no)
+			(effects
+				(font
+					(size 1.27 1.27)
+				)
+			)
+		)
+		(property "Value" "OCT 1x6h"
+			(at 103.505 48.26 0)
+			(show_name no)
+			(do_not_autoplace no)
+			(effects
+				(font
+					(size 1.27 1.27)
+				)
+			)
+		)
+		(property "Footprint" "Connector_PinHeader_2.54mm:PinHeader_1x06_P2.54mm_Vertical"
+			(at 102.87 55.88 0)
+			(hide yes)
+			(show_name no)
+			(do_not_autoplace no)
+			(effects
+				(font
+					(size 1.27 1.27)
+				)
+			)
+		)
+		(property "Datasheet" ""
+			(at 102.87 55.88 0)
+			(hide yes)
+			(show_name no)
+			(do_not_autoplace no)
+			(effects
+				(font
+					(size 1.27 1.27)
+				)
+			)
+		)
+		(property "Description" "Generic connector, single row, 01x06, script generated"
+			(at 102.87 55.88 0)
+			(hide yes)
+			(show_name no)
+			(do_not_autoplace no)
+			(effects
+				(font
+					(size 1.27 1.27)
+				)
+			)
+		)
+		(pin "4"
+		)
+		(pin "5"
+		)
+		(pin "6"
+		)
+		(pin "3"
+		)
+		(pin "1"
+		)
+		(pin "2"
+		)
+		(instances
+			(project "VCO 2"
+				(path "/eb1652b6-57da-4a0e-88a4-449907a19840/2395376b-3fab-44b6-8171-4759de5684a3"
+					(reference "J22")
+					(unit 1)
+				)
+			)
+		)
+	)
+	(symbol
 		(lib_id "power:GND")
 		(at 261.62 72.39 0)
@@
 	)
 	(symbol
+		(lib_id "power:GND")
+		(at 118.11 66.04 0)
+		(unit 1)
+		(body_style 1)
+		(exclude_from_sim no)
+		(in_bom yes)
+		(on_board yes)
+		(in_pos_files yes)
+		(dnp no)
+		(fields_autoplaced yes)
+		(property "Reference" "#PWR044"
+			(at 118.11 72.39 0)
+			(hide yes)
+			(show_name no)
+			(do_not_autoplace no)
+			(effects
+				(font
+					(size 1.27 1.27)
+				)
+			)
+		)
+		(property "Value" "GND"
+			(at 118.11 71.12 0)
+			(show_name no)
+			(do_not_autoplace no)
+			(effects
+				(font
+					(size 1.27 1.27)
+				)
+			)
+		)
+		(property "Footprint" ""
+			(at 118.11 66.04 0)
+			(hide yes)
+			(show_name no)
+			(do_not_autoplace no)
+			(effects
+				(font
+					(size 1.27 1.27)
+				)
+			)
+		)
+		(property "Datasheet" ""
+			(at 118.11 66.04 0)
+			(hide yes)
+			(show_name no)
+			(do_not_autoplace no)
+			(effects
+				(font
+					(size 1.27 1.27)
+				)
+			)
+		)
+		(property "Description" "Power symbol creates a global label with name \"GND\" , ground"
+			(at 118.11 66.04 0)
+			(hide yes)
+			(show_name no)
+			(do_not_autoplace no)
+			(effects
+				(font
+					(size 1.27 1.27)
+				)
+			)
+		)
+		(pin "1"
+		)
+		(instances
+			(project "VCO 2"
+				(path "/eb1652b6-57da-4a0e-88a4-449907a19840/2395376b-3fab-44b6-8171-4759de5684a3"
+					(reference "#PWR044")
+					(unit 1)
+				)
+			)
+		)
+	)
+	(symbol
 		(lib_id "Connector_Audio:AudioJack2_SwitchT")
 		(at 25.4 134.62 0)
@@
 					(unit 1)
 				)
-			)
-		)
-	)
-	(symbol
-		(lib_id "Connector:Conn_01x07_Pin")
-		(at 102.87 58.42 0)
-		(unit 1)
-		(body_style 1)
-		(exclude_from_sim no)
-		(in_bom yes)
-		(on_board yes)
-		(in_pos_files yes)
-		(dnp no)
-		(property "Reference" "J17"
-			(at 103.505 45.72 0)
-			(show_name no)
-			(do_not_autoplace no)
-			(effects
-				(font
-					(size 1.27 1.27)
-				)
-			)
-		)
-		(property "Value" "OCT_SW 1x7h"
-			(at 103.505 48.26 0)
-			(show_name no)
-			(do_not_autoplace no)
-			(effects
-				(font
-					(size 1.27 1.27)
-				)
-			)
-		)
-		(property "Footprint" "Connector_PinHeader_2.54mm:PinHeader_1x07_P2.54mm_Vertical"
-			(at 102.87 58.42 0)
-			(hide yes)
-			(show_name no)
-			(do_not_autoplace no)
-			(effects
-				(font
-					(size 1.27 1.27)
-				)
-			)
-		)
-		(property "Datasheet" ""
-			(at 102.87 58.42 0)
-			(hide yes)
-			(show_name no)
-			(do_not_autoplace no)
-			(effects
-				(font
-					(size 1.27 1.27)
-				)
-			)
-		)
-		(property "Description" "Generic connector, single row, 01x07, script generated"
-			(at 102.87 58.42 0)
-			(hide yes)
-			(show_name no)
-			(do_not_autoplace no)
-			(effects
-				(font
-					(size 1.27 1.27)
-				)
-			)
-		)
-		(pin "7"
-		)
-		(pin "4"
-		)
-		(pin "1"
-		)
-		(pin "5"
-		)
-		(pin "2"
-		)
-		(pin "6"
-		)
-		(pin "3"
-		)
-		(instances
-			(project "VCO 2"
-				(path "/eb1652b6-57da-4a0e-88a4-449907a19840/2395376b-3fab-44b6-8171-4759de5684a3"
-					(reference "J17")
-					(unit 1)
-				)

Commit message: Updated switch footprint to use imported footprint
Parts:
- SW1: footprint Switch:SW_Toggle_Blue_wSlots -> Mini-Switch:2MS1T1-M2_DYW
Changed lines of the file:
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@@
 			)
 		)
-		(property "Footprint" "Switch:SW_Toggle_Blue_wSlots"
+		(property "Footprint" "Mini-Switch:2MS1T1-M2_DYW"
 			(at 198.12 107.95 0)
 			(hide yes)

Commit message: Fixed switches, added new FPs and symbols.
Parts:
- removed SW2: SW_Rotary_1x6_MP, Rotary Switch:SR1712F-0106-20F0A-N9-N-027_ATW, symbol Switch:SW_Rotary_1x6_MP
- added U5: RS1702A0A-HA1, Rotary 6-Way SW:rotary-6-way-sw, symbol Rotary Switch:SR1712F-0106-20F0A-N9-N-027
- SW1: footprint Mini-Switch:2MS1T1-M2_DYW -> sub-miniture-SPDT:Sub-miniture SPDT
Connections:
- net GND: now also U5.7
- net at J22.1 (Pin_1): now also U5.2
- net at J22.2 (Pin_2): now also U5.3
- net at J22.3 (Pin_3): now also U5.4
- net at J22.4 (Pin_4): now also U5.5
- net at J22.5 (Pin_5): now also U5.6
- net at J22.6 (Pin_6): now also U5.1
- no-connect marks 10 -> 12

Commit message: Corrected connections for levels and octave switch
Connections:
- net GND: now also RV2.1, RV3.1; no longer RV2.3, RV3.3
- net at J22.1 (Pin_1): now also U5.1; no longer U5.2
- net at J22.2 (Pin_2): now also U5.6; no longer U5.3
- net at J22.3 (Pin_3): now also U5.5; no longer U5.4
- net at J22.4 (Pin_4): now also U5.4; no longer U5.5
- net at J22.5 (Pin_5): now also U5.3; no longer U5.6
- net at J22.6 (Pin_6): now also U5.2; no longer U5.1
- net at J12.T: now also RV3.3; no longer RV3.1
- net at J13.T: now also RV2.3; no longer RV2.1
Other:
- note added: "1.3"
- moved on the sheet: RV2, RV3
Changed lines of the file:
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@@
 		)
 	)
+	(text "1.3"
+		(exclude_from_sim no)
+		(at 270.51 193.294 0)
+		(effects
+			(font
+				(size 1.27 1.27)
+			)
+		)
+	)
 	(junction
 		(at 196.85 73.66)
@@
 	(wire
 		(pts
-			(xy 107.95 63.5) (xy 113.03 63.5)
-		)
-		(stroke
-			(width 0)
-			(type default)
-		)
-	)
-	(wire
-		(pts
 			(xy 213.36 105.41) (xy 213.36 116.84)
 		)
@@
 	(wire
 		(pts
+			(xy 107.95 63.5) (xy 113.03 63.5)
+		)
+		(stroke
+			(width 0)
+			(type default)
+		)
+	)
+	(wire
+		(pts
 			(xy 30.48 110.49) (xy 33.02 110.49)
 		)
@@
 	)
 	(symbol
-		(lib_id "Connector:Conn_01x06_Pin")
-		(at 102.87 55.88 0)
-		(unit 1)
-		(body_style 1)
-		(exclude_from_sim no)
-		(in_bom yes)
-		(on_board yes)
-		(in_pos_files yes)
-		(dnp no)
-		(fields_autoplaced yes)
-		(property "Reference" "J22"
-			(at 103.505 45.72 0)
-			(show_name no)
-			(do_not_autoplace no)
-			(effects
-				(font
-					(size 1.27 1.27)
-				)
-			)
-		)
-		(property "Value" "OCT 1x6h"
-			(at 103.505 48.26 0)
-			(show_name no)
-			(do_not_autoplace no)
-			(effects
-				(font
-					(size 1.27 1.27)
-				)
-			)
-		)
-		(property "Footprint" "Connector_PinHeader_2.54mm:PinHeader_1x06_P2.54mm_Vertical"
-			(at 102.87 55.88 0)
-			(hide yes)
-			(show_name no)
-			(do_not_autoplace no)
-			(effects
-				(font
-					(size 1.27 1.27)
-				)
-			)
-		)
-		(property "Datasheet" ""
-			(at 102.87 55.88 0)
-			(hide yes)
-			(show_name no)
-			(do_not_autoplace no)
-			(effects
-				(font
-					(size 1.27 1.27)
-				)
-			)
-		)
-		(property "Description" "Generic connector, single row, 01x06, script generated"
-			(at 102.87 55.88 0)
-			(hide yes)
-			(show_name no)
-			(do_not_autoplace no)
-			(effects
-				(font
-					(size 1.27 1.27)
-				)
-			)
-		)
-		(pin "4"
-		)
-		(pin "5"
-		)
-		(pin "6"
-		)
-		(pin "3"
-		)
-		(pin "1"
-		)
-		(pin "2"
-		)
-		(instances
-			(project "VCO 2"
-				(path "/eb1652b6-57da-4a0e-88a4-449907a19840/2395376b-3fab-44b6-8171-4759de5684a3"
-					(reference "J22")
-					(unit 1)
-				)
-			)
-		)
-	)
-	(symbol
 		(lib_id "power:GND")
 		(at 261.62 72.39 0)
@@
 	(symbol
 		(lib_id "Device:R_Potentiometer")
-		(at 45.72 113.03 90)
+		(at 45.72 113.03 270)
+		(mirror x)
 		(unit 1)
 		(body_style 1)
@@
 		(in_pos_files yes)
 		(dnp no)
-		(fields_autoplaced yes)
 		(property "Reference" "RV2"
 			(at 45.72 116.84 90)
@@
 	)
 	(symbol
-		(lib_id "Device:R_Potentiometer")
-		(at 44.45 48.26 90)
+		(lib_id "Connector:Conn_01x06_Pin")
+		(at 102.87 58.42 0)
+		(mirror x)
 		(unit 1)
 		(body_style 1)
@@
 		(dnp no)
 		(fields_autoplaced yes)
+		(property "Reference" "J22"
+			(at 103.505 45.72 0)
+			(show_name no)
+			(do_not_autoplace no)
+			(effects
+				(font
+					(size 1.27 1.27)
+				)
+			)
+		)
+		(property "Value" "OCT 1x6h"
+			(at 103.505 48.26 0)
+			(show_name no)
+			(do_not_autoplace no)
+			(effects
+				(font
+					(size 1.27 1.27)
+				)
+			)
+		)
+		(property "Footprint" "Connector_PinHeader_2.54mm:PinHeader_1x06_P2.54mm_Vertical"
+			(at 102.87 58.42 0)
+			(hide yes)
+			(show_name no)
+			(do_not_autoplace no)
+			(effects
+				(font
+					(size 1.27 1.27)
+				)
+			)
+		)
+		(property "Datasheet" ""
+			(at 102.87 58.42 0)
+			(hide yes)
+			(show_name no)
+			(do_not_autoplace no)
+			(effects
+				(font
+					(size 1.27 1.27)
+				)
+			)
+		)
+		(property "Description" "Generic connector, single row, 01x06, script generated"
+			(at 102.87 58.42 0)
+			(hide yes)
+			(show_name no)
+			(do_not_autoplace no)
+			(effects
+				(font
+					(size 1.27 1.27)
+				)
+			)
+		)
+		(pin "4"
+		)
+		(pin "5"
+		)
+		(pin "6"
+		)
+		(pin "3"
+		)
+		(pin "1"
+		)
+		(pin "2"
+		)
+		(instances
+			(project "VCO 2"
+				(path "/eb1652b6-57da-4a0e-88a4-449907a19840/2395376b-3fab-44b6-8171-4759de5684a3"
+					(reference "J22")
+					(unit 1)
+				)
+			)
+		)
+	)
+	(symbol
+		(lib_id "Device:R_Potentiometer")
+		(at 44.45 48.26 270)
+		(mirror x)
+		(unit 1)
+		(body_style 1)
+		(exclude_from_sim no)
+		(in_bom yes)
+		(on_board yes)
+		(in_pos_files yes)
+		(dnp no)
 		(property "Reference" "RV3"
 			(at 44.45 52.07 90)
