File: VCO 2.kicad_pcb (KiCad board)
At the start: 2 copper layers, 185.7 x 142.5 mm, 132 parts, among them J1 OUT 1x4s, J10 IN 1x6h, J11 SYNC, J12 PWM, J13 CV, J14 1VOct, J15 FM, J17 OCT 1x6s, J18 CV 1x6s, J19 CV 1x6h, J2 SQR, J20 LED 1x2s, J21 LED 1x2h, J22 OCT 1x6h, J3 OUT 1x4h, J4 SAW, J5 TRI, J6 SIN, J7 CTRL 1x8h, J8 CTRL 1x8s, J85 Eurorack 2x8hs, J9 IN 1x6s, Q1 2N3904, Q2 2N3904, SW1 SW_SPDT, U1 CEM3340, U2 TL074, U3 TL074, U4 LM336Z-2.5, U5 RS1702A0A-HA1

Commit message: Fixed oct selector and updated gnd islands on main
Parts:
- moved R19 0.87 mm to (66.6, 70.0)
Connections:
- U5 pad 1: Net-(J22-Pin_1) -> Net-(J22-Pin_6)
- U5 pad 2: Net-(J22-Pin_6) -> GND
- U5 pad 7: GND -> Net-(J22-Pin_1)
Routing:
- net Net-(J22-Pin_1): track 28.8 -> 7.36 mm
- net Net-(J22-Pin_6): track 51.8 -> 46.2 mm
- net Net-(J22-Pin_4): track 31.1 -> 32.2 mm
- net Net-(J22-Pin_5): track 35.7 -> 36.8 mm
- net Net-(J22-Pin_3): track 26.2 -> 27.2 mm
- net Net-(J17-Pin_6): track 27.4 -> 28.0 mm
- net GND: track 5.83 -> 5.78 mm, vias 22 -> 20
Other:
- board text added: "VCO2 - Controls Ver: 1.4 Nigel Daniels 2026"
- board text added: "VCO2 - Front Panel Ver: 1.4 Nigel Daniels 2026"
- board text added: "VCO2 - Main Board Ver: 1.4 Nigel Daniels 2026"
- board text removed: "VCO2 - Controls Ver: 1.3 Nigel Daniels 2026"
- board text removed: "VCO2 - Front Panel Ver: 1.3 Nigel Daniels 2026"
- board text removed: "VCO2 - Main Board Ver: 1.3 Nigel Daniels 2026"

Commit message: Updated unflipped connector on control
Parts:
- J22: moved to B.Cu
- turned J22 to 180 degrees

Commit message: Reversed power oct. selector and flipped power in
Parts:
- moved J85 17.9 mm to (80.1, 127.8), turned to 0 degrees
- moved D10 10.8 mm to (76.2, 131.8)
- moved D11 10.6 mm to (65.5, 121.1)
- moved C20 8.10 mm to (52.5, 120.5)
- moved C21 7.97 mm to (52.4, 133.5)
- moved C19 7.13 mm to (59.6, 131.2)
- moved C18 7.12 mm to (59.6, 121.5)
- moved R74 5.77 mm to (69.4, 127.3)
- moved R73 5.72 mm to (74.9, 125.5)
- moved R31 0.10 mm to (37.6, 56.4)
Connections:
- J17 pad 1: REF -> Net-(J17-Pin_1)
- J17 pad 5: Net-(J17-Pin_5) -> REF
- R27 pad 1: REF -> Net-(J17-Pin_1)
- R30 pad 2: Net-(J17-Pin_5) -> REF
- R31 pad 1: Net-(J17-Pin_5) -> Net-(J17-Pin_1)
- U3 pad 5: Net-(J17-Pin_5) -> Net-(J17-Pin_1)
Routing:
- net Net-(J17-Pin_1): track 0.00 -> 36.2 mm
- net Net-(J17-Pin_5): track 27.1 -> 0.00 mm
- net +12v: track 270.6 -> 292.2 mm
- net REF: track 89.5 -> 98.3 mm
- net -12V: track 15.4 -> 9.66 mm
- net +12V: track 15.6 -> 10.1 mm
- net Net-(D11-K): track 4.74 -> 8.66 mm
- net Net-(D10-A): track 8.66 -> 4.74 mm
- net Net-(J18-Pin_1): track 42.5 -> 41.3 mm
- net -12v: track 190.2 -> 189.5 mm
- net GND: vias 20 -> 21
Other:
- board text added: "1.5"
- board text added: "VCO2 - Controls Ver: 1.5 Nigel Daniels 2026"
- board text added: "VCO2 - Front Panel Ver: 1.5 Nigel Daniels 2026"
- board text added: "VCO2 - Main Board Ver: 1.5 Nigel Daniels 2026"
- board text removed: "1.3"
- board text removed: "Apr 2026"
- board text removed: "VCO2 - Controls Ver: 1.4 Nigel Daniels 2026"
- board text removed: "VCO2 - Front Panel Ver: 1.4 Nigel Daniels 2026"
- board text removed: "VCO2 - Main Board Ver: 1.4 Nigel Daniels 2026"

Commit message: Reverted power connection switch and updated schematics.
Connections:
- J17 pad 1: Net-(J17-Pin_1) -> REF
- J17 pad 5: REF -> Net-(J17-Pin_5)
- R27 pad 1: Net-(J17-Pin_1) -> REF
- R30 pad 2: REF -> Net-(J17-Pin_5)
- R31 pad 1: Net-(J17-Pin_1) -> Net-(J17-Pin_5)
- U3 pad 5: Net-(J17-Pin_1) -> Net-(J17-Pin_5)
Routing:
- net Net-(J17-Pin_1): track 36.2 -> 0.00 mm
- net Net-(J17-Pin_5): track 0.00 -> 27.6 mm
- net REF: track 98.3 -> 89.4 mm
Other:
- board text added: "1.4"
- board text added: "VCO2 - Controls Ver: 1.4 Nigel Daniels 2026"
- board text added: "VCO2 - Front Panel Ver: 1.4 Nigel Daniels 2026"
- board text added: "VCO2 - Main Board Ver: 1.4 Nigel Daniels 2026"
- board text removed: "1.5"
- board text removed: "VCO2 - Controls Ver: 1.5 Nigel Daniels 2026"
- board text removed: "VCO2 - Front Panel Ver: 1.5 Nigel Daniels 2026"
- board text removed: "VCO2 - Main Board Ver: 1.5 Nigel Daniels 2026"
