File: VCO 2.kicad_sch (KiCad schematic)
At the start: 99 parts, among them J1 OUT 1x4s, J17 OCT 1x6s, J18 CV 1x6s, J20 LED 1x2s, J8 CTRL 1x8s, J85 Eurorack 2x8hs, J9 IN 1x6s, Q1 2N3904, Q2 2N3904, U1 CEM3340, U2 TL074, U3 TL074, U4 LM336Z-2.5

Commit message: Reverted power connection switch and updated schematics.
Connections:
- net REF: now also J17.1 (Pin_1), R27.1; no longer J17.5 (Pin_5), R30.2
- net at R31.1, U3.5 (+): now also J17.5 (Pin_5), R30.2; no longer J17.1 (Pin_1), R27.1
